Commit message: Add files via upload

File: doggybot_description/urdf/leg_wheel.xacro (robot description, xacro)
@@ -4,5 +4,5 @@
        <inertial>
           <origin xyz="0 0 0" rpy="0 0 0"/>
-          <mass value="0.030"/>
+          <mass value="0.130"/>
           <inertia ixx="1.75e-5" ixy="0" ixz="0" iyy="1.75e-5" iyz="0" izz="1.75e-5"/>
        </inertial>
