Commit message: gazebo configuration
Added camera sensor, added teleoperation GUI in gazebo, urdf physical parameters

File: doggybot_description/urdf/body.xacro (robot description, xacro)
@@ -1,4 +1,5 @@
 <robot xmlns:xacro="http://www.ros.org/wiki/xacro"  name="body">
   <xacro:include filename="$(find doggybot_description)/urdf/leg_wheel.xacro" />
+  <xacro:include filename="$(find doggybot_description)/urdf/sensors.xacro" />
   <xacro:macro name="base">
   <link name="head_link" >
@@ -24,4 +25,26 @@
            </inertial>
      </link>
+  <link name="tail_link" >
+          <visual>
+                 <origin xyz="0 0 0" rpy="0 0 0"/>
+                 <geometry>
+                         <box size="0.1 0.1 0.3"/>
+                 </geometry>
+                 <material name="Head_Blue">
+                         <color rgba="${30/255} ${144/255} ${255/255} 0.8"/>
+                 </material>
+           </visual>
+           <collision>
+                  <origin xyz="0 0 0" rpy="0 0 0"/>
+                  <geometry>
+                          <box size="0.1 0.1 0.3"/>
+                  </geometry>
+           </collision>
+           <inertial>
+                   <origin xyz="0 0 ${0.5*0.5}" rpy="0 0 0"/>
+                   <mass value="0.01"/>
+                   <inertia ixx="6.0e-4" ixy="0" ixz="0" iyy="6.0e-4" iyz="0" izz="6.0e-4"/>
+           </inertial>
+     </link>
   <link name="base_link" >
           <visual>
@@ -42,5 +65,5 @@
            <inertial>
                    <origin xyz="0 0 ${0.5*0.5}" rpy="0 0 0"/>
-                   <mass value="0.180"/>
+                   <mass value="0.280"/>
                    <inertia ixx="6.0e-4" ixy="0" ixz="0" iyy="6.0e-4" iyz="0" izz="6.0e-4"/>
            </inertial>
@@ -51,15 +74,26 @@
       <origin xyz="0.0 0.35 0.3" rpy="0 0 0"/>
     </joint>
+    <joint name="tail" type="fixed">
+      <parent link="base_link"/>
+      <child  link="tail_link"/>
+      <origin xyz="0.0 -0.45 0.1" rpy="-0.5 0.0 0"/>
+    </joint>
+    <joint name="camera_mount" type="fixed">
+      <parent link="head_link"/>
+      <child  link="rgb_camera"/>
+      <origin xyz="0.0 0.19 0.02" rpy="0 0 ${3.1415/2}"/>
+    </joint>
+   <xacro:camera/>
    <xacro:leg prefix="front_left">
-      <origin xyz="-0.3 0.35 -0.3" rpy="${-3.1415/2} 0 ${-3.1415/2}"/>
+      <origin xyz="-0.3 0.35 -0.3" rpy="${-3.1415/2-0.2} 0.2 ${-3.1415/2}"/>
    </xacro:leg>
    <xacro:leg prefix="front_right">
-      <origin xyz="0.3 0.35 -0.3" rpy="${-3.1415/2} 0 ${-3.1415/2}"/>
+      <origin xyz="0.3 0.35 -0.3" rpy="${-3.1415/2+0.2} 0.2 ${-3.1415/2}"/>
    </xacro:leg>
    <xacro:leg prefix="back_left">
-      <origin xyz="-0.3 -0.35 -0.3" rpy="${-3.1415/2} 0 ${-3.1415/2}"/>
+      <origin xyz="-0.3 -0.35 -0.3" rpy="${-3.1415/2-0.2} -0.2 ${-3.1415/2}"/>
    </xacro:leg>
    <xacro:leg prefix="back_right">
-      <origin xyz="0.3 -0.35 -0.3" rpy="${-3.1415/2} 0 ${-3.1415/2}"/>
+      <origin xyz="0.3 -0.35 -0.3" rpy="${-3.1415/2+0.2} -0.2 ${-3.1415/2}"/>
    </xacro:leg>
   </xacro:macro>

File: doggybot_description/urdf/leg_wheel.xacro (robot description, xacro)
@@ -50,7 +50,7 @@
 	<origin xyz="0 0 0" rpy="${3.1415/2} 0 0"/>
 	<geometry>
-	  <cylinder length="0.05" radius="0.2"/>
+	  <cylinder length="0.1" radius="0.2"/>
 	</geometry>
-	<material name="blue">
+	<material name="wheel_red">
 	  <color rgba="${255/255} ${0/255} ${0/255}  0.8"/>
 	</material>
@@ -59,9 +59,27 @@
 	<origin xyz="0 0 0" rpy="${3.1415/2} 0 0"/>
 	<geometry>
-	  <cylinder length="0.05" radius="0.2"/>
+	  <cylinder length="0.0001" radius="0.2"/>
 	</geometry>
 	<material name="blue">
 	  <color rgba="0.0 1.0 0.0 0.5"/>
 	</material>
+	<surface>
+    <friction>
+      <ode>
+        <mu>5.0</mu>       <!-- strong forward friction -->
+        <mu2>2.0</mu2>     <!-- slightly less lateral grip -->
+      </ode>
+    </friction>
+    <bounce>
+      <restitution_coefficient>0.05</restitution_coefficient>
+      <threshold>0.1</threshold>
+    </bounce>
+    <contact>
+      <soft_cfm>1e-5</soft_cfm>   <!-- slight softness -->
+      <soft_erp>0.6</soft_erp>
+      <kp>50000</kp>             <!-- stiffer than soft material -->
+      <kd>5.0</kd>
+    </contact>
+  </surface>
       </collision>
      </link>

Commit message: Add files via upload

File: doggybot_description/urdf/body.xacro (robot description, xacro)
@@ -25,4 +25,7 @@
            </inertial>
      </link>
+  <link name="body_link" >
+    <origin xyz="0 0 0" rpy="0 0 0"/>
+  </link>
   <link name="tail_link" >
           <visual>
@@ -69,4 +72,9 @@
            </inertial>
      </link>
+    <joint name="trans" type="fixed">
+      <parent link="body_link"/>
+      <child  link="base_link"/>
+      <origin xyz="0.0 0.0 0.0" rpy="0 0 -${3.1415/2}"/>
+    </joint>
     <joint name="head" type="fixed">
       <parent link="base_link"/>
@@ -79,4 +87,7 @@
       <origin xyz="0.0 -0.45 0.1" rpy="-0.5 0.0 0"/>
     </joint>
+    <xacro:lidar_sensor>
+     <origin xyz="0 0.1 -0.2" rpy="0 0 ${3.1415/2}"/>
+    </xacro:lidar_sensor>
     <joint name="camera_mount" type="fixed">
       <parent link="head_link"/>
@@ -86,14 +97,14 @@
    <xacro:camera/>
    <xacro:leg prefix="front_left">
-      <origin xyz="-0.3 0.35 -0.3" rpy="${-3.1415/2-0.2} 0.2 ${-3.1415/2}"/>
+      <origin xyz="-0.3 0.35 -0.3" rpy="${-3.1415/2-0.3} 0.2 ${-3.1415/2}"/>
    </xacro:leg>
    <xacro:leg prefix="front_right">
-      <origin xyz="0.3 0.35 -0.3" rpy="${-3.1415/2+0.2} 0.2 ${-3.1415/2}"/>
+      <origin xyz="0.3 0.35 -0.3" rpy="${-3.1415/2+0.3} 0.2 ${-3.1415/2}"/>
    </xacro:leg>
    <xacro:leg prefix="back_left">
-      <origin xyz="-0.3 -0.35 -0.3" rpy="${-3.1415/2-0.2} -0.2 ${-3.1415/2}"/>
+      <origin xyz="-0.3 -0.35 -0.3" rpy="${-3.1415/2-0.3} -0.2 ${-3.1415/2}"/>
    </xacro:leg>
    <xacro:leg prefix="back_right">
-      <origin xyz="0.3 -0.35 -0.3" rpy="${-3.1415/2+0.2} -0.2 ${-3.1415/2}"/>
+      <origin xyz="0.3 -0.35 -0.3" rpy="${-3.1415/2+0.3} -0.2 ${-3.1415/2}"/>
    </xacro:leg>
   </xacro:macro>

File: doggybot_description/urdf/leg_wheel.xacro (robot description, xacro)
@@ -36,6 +36,6 @@
       <parent link="${prefix}_leg"/>
       <child  link="${prefix}_wheel"/>
-      <origin xyz="0.0 0.2 0" rpy="${-3.1415/2} 0 ${-3.1415/2}"/>
-      <axis xyz="0 1 0"/>
+      <origin xyz="0.0 0.2 0" rpy="0 ${3.1415/2} 0"/>
+      <axis xyz="1 0 0"/>
     </joint>
   </xacro:macro>
@@ -48,5 +48,5 @@
        </inertial>
        <visual>
-	<origin xyz="0 0 0" rpy="${3.1415/2} 0 0"/>
+	<origin xyz="0 0 0" rpy="${3.1415/2} 0 ${3.1415/2}"/>
 	<geometry>
 	  <cylinder length="0.1" radius="0.2"/>
@@ -57,7 +57,7 @@
       </visual>
       <collision>
-	<origin xyz="0 0 0" rpy="${3.1415/2} 0 0"/>
+	<origin xyz="0 0 0" rpy="${3.1415/2} 0 ${3.1415/2}"/>
 	<geometry>
-	  <cylinder length="0.0001" radius="0.2"/>
+	  <sphere radius="0.2"/>
 	</geometry>
 	<material name="blue">
@@ -67,6 +67,6 @@
     <friction>
       <ode>
-        <mu>5.0</mu>       <!-- strong forward friction -->
-        <mu2>2.0</mu2>     <!-- slightly less lateral grip -->
+        <mu>1.0</mu>       <!-- strong forward friction -->
+        <mu2>0.1</mu2>     <!-- slightly less lateral grip -->
       </ode>
     </friction>

File: doggybot_description/urdf/sensors.xacro (robot description, xacro)
@@ -47,3 +47,54 @@
     </gazebo>
   </xacro:macro>
+  <xacro:macro name="lidar_sensor" params="*origin">
+     <link name="lidar_link">
+          <visual>
+                 <origin xyz="0 0 0" rpy="${3.1415/2} 0 ${3.1415/2}"/>
+                 <material name="Red">
+                         <color rgba="1.0 0.0 0.0 0.5"/>
+                 </material>
+           </visual>
+           <collision>
+                 <origin xyz="0 0 0" rpy="${3.1415/2} 0 ${3.1415/2}"/>
+                  <material name="Red">
+                         <color rgba="1.0 0.0 0.0 0.5"/>
+                  </material>
+           </collision>
+     </link>
+     <joint name="lidar_joint" type="fixed">
+       <parent link="head_link"/>
+       <child link="lidar_link"/>
+       <xacro:insert_block name="origin" />
+     </joint>
+    <gazebo reference="lidar_link" >
+      <sensor name="lidar" type="gpu_lidar">
+        <topic> lidar_scan </topic>
+        <update_rate>100</update_rate>
+        <ignition_frame_id>lidar_link</ignition_frame_id>
+        <ray>
+          <scan>
+            <horizontal>
+              <samples>300</samples>
+              <resolution>1</resolution>
+              <min_angle>${-3.1415/2}</min_angle>
+              <max_angle>${3.1415/2}</max_angle>
+            </horizontal>
+            <vertical>
+              <samples>30</samples>
+              <resolution>1</resolution>
+              <min_angle>-${3.1415/2-1}</min_angle>
+              <max_angle>0.2618</max_angle>
+            </vertical>
+          </scan>
+          <range>
+            <min>0.02</min>
+            <max>30.0</max>
+            <resolution>100</resolution>
+          </range>
+        </ray>
+        <alwaysOn>1</alwaysOn>
+        <visualize>true</visualize>
+      </sensor>
+    </gazebo>
+  </xacro:macro>
 </robot>
